File: pcb-files/echo.kicad_pcb (KiCad board)
At the start: 2 copper layers, 93.6 x 80.2 mm, 11 parts, among them SW1 SW_Push, SW3 SW_Push, SW4 SW_Push, U1 XIAO-RP2040-SMD

Commit message: added kicad files + gerbers
Parts:
- added REF**: MountingHole_2.2mm_M2, MountingHole:MountingHole_2.2mm_M2, F.Cu at (119.8, 106.2)
- added REF**: MountingHole_2.2mm_M2, MountingHole:MountingHole_2.2mm_M2, F.Cu at (119.6, 35.6)
- added REF**: MountingHole_2.2mm_M2, MountingHole:MountingHole_2.2mm_M2, F.Cu at (36.8, 35.8)
- added REF**: MountingHole_2.2mm_M2, MountingHole:MountingHole_2.2mm_M2, F.Cu at (36.8, 106.2)
Routing:
- net GND: track 193.2 -> 6.47 mm
- added copper zone on B.Cu, net GND
- added copper zone on F.Cu, net GND
